Commit message: add modified urdf

File: digit_model.urdf (robot description, URDF)
Before this commit: robot digit, 25 links, 24 joints
Links:
- link left_elbow: mass 0.550582 -> 5.550582
- link right_elbow: mass 0.550582 -> 5.550582

Commit message: added 1kg 2kg cases

File: digit_model.urdf (robot description, URDF)
Before this commit: robot digit, 25 links, 24 joints
Links:
- link left_elbow: mass 5.550582 -> 1.050582
- link right_elbow: mass 5.550582 -> 1.050582
